File: gocon2026badge/gocon2026badge/gocon2026badge.kicad_pcb (KiCad board)
At the start: 2 copper layers, 100 x 100 mm, 34 parts, among them SW1 SW_PUSH, SW2 SW_PUSH, SW3 SW_PUSH, SW4 SW_PUSH, SW5 SW_PUSH, SW6 SW_PUSH, U1 rp2040-zero, U2 ST7789-1.54TFT-SPI, U3 GROVE_I2C_UART, U4 PCM510x, U5 GROVE_I2C_UART

Commit message: Update gocon2026badge
Parts:
- removed SW6: SW_PUSH, sglib:SW_PUSH_6mm_H5mm-b
- removed U3, U5: GROVE_I2C_UART, sglib:grove-horizontal-b
- removed U4: PCM510x, sglib:PinHeader_1x06_P2.54mm_Vertical-b
Routing:
- net VCC: track 414.6 -> 265.8 mm, vias 5 -> 3
- net I2C1_SCL: track 102.4 -> 0.00 mm, vias 2 -> 0
- net I2C1_SDA: track 99.4 -> 0.00 mm, vias 2 -> 0
- net I2C0_SDA: track 99.1 -> 0.00 mm, vias 2 -> 0
- net I2C0_SCL: track 93.6 -> 0.00 mm, vias 2 -> 0
- net GND: track 491.1 -> 400.2 mm, vias 6 -> 2
- net BTN_B: track 60.5 -> 0.00 mm
- net PCM510x_LRCK: track 50.8 -> 0.00 mm
- net PCM510x_DIN: track 44.2 -> 0.00 mm
- net PCM510x_BCK: track 44.2 -> 0.00 mm
